File: sensorboard.sch (EAGLE design)
At the start: 20 parts, among them IC1 LD117AS18TR, K2 JTN-PCB-DC18V, Q1 BC639, Q2 BC639

Commit message: Add files via upload
Version2 (88 X 59.50)
Parts:
- removed JP3: (no value), pinhead:PINHD-1X2
- added X2: (no value), con-ptr500:AK500/2
Connections:
- net GND: now also X2-1.KL; no longer JP3.2
- net VDD3V3: now also X2-2.KL; no longer JP3.1
Changed lines of the file:
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@@
 <part name="K2" library="relay" library_urn="urn:adsk.eagle:library:339" deviceset="JT?-*" device="N-PCB" package3d_urn="urn:adsk.eagle:package:24456/1" technology="DC18V"/>
 <part name="JP1" library="pinhead" library_urn="urn:adsk.eagle:library:325" deviceset="PINHD-1X7" device="" package3d_urn="urn:adsk.eagle:package:22477/2"/>
-<part name="JP3" library="pinhead" library_urn="urn:adsk.eagle:library:325" deviceset="PINHD-1X2" device="" package3d_urn="urn:adsk.eagle:package:22435/2"/>
 <part name="X3" library="con-ptr500" library_urn="urn:adsk.eagle:library:181" deviceset="AK500/3" device="" package3d_urn="urn:adsk.eagle:package:9883/1"/>
+<part name="X2" library="con-ptr500" library_urn="urn:adsk.eagle:library:181" deviceset="AK500/2" device="" package3d_urn="urn:adsk.eagle:package:9880/1"/>
 </parts>
 <sheets>
@@
 <attribute name="VALUE" x="19.05" y="88.9" size="1.778" layer="96" rot="R180"/>
 </instance>
-<instance part="JP3" gate="G$1" x="76.2" y="20.32" smashed="yes">
-<attribute name="NAME" x="69.85" y="26.035" size="1.778" layer="95"/>
-<attribute name="VALUE" x="69.85" y="15.24" size="1.778" layer="96"/>
-</instance>
 <instance part="X3" gate="-1" x="170.18" y="35.56" smashed="yes" rot="R180">
 <attribute name="NAME" x="171.45" y="34.671" size="1.778" layer="95"/>
@@
 <attribute name="NAME" x="171.45" y="44.831" size="1.778" layer="95"/>
 <attribute name="VALUE" x="173.99" y="49.403" size="1.778" layer="96" rot="R180"/>
+</instance>
+<instance part="X2" gate="-1" x="71.12" y="20.32" smashed="yes" rot="R180">
+<attribute name="NAME" x="72.39" y="19.431" size="1.778" layer="95"/>
+</instance>
+<instance part="X2" gate="-2" x="71.12" y="25.4" smashed="yes" rot="R180">
+<attribute name="NAME" x="72.39" y="24.511" size="1.778" layer="95"/>
+<attribute name="VALUE" x="74.93" y="29.083" size="1.778" layer="96" rot="R180"/>
 </instance>
 </instances>
@@
 </segment>
 <segment>
-<pinref part="JP3" gate="G$1" pin="2"/>
-<wire x1="73.66" y1="20.32" x2="66.04" y2="20.32" width="0.1524" layer="91"/>
-<label x="60.96" y="20.32" size="1.778" layer="95"/>
+<pinref part="X2" gate="-1" pin="KL"/>
+<wire x1="66.04" y1="20.32" x2="58.42" y2="20.32" width="0.1524" layer="91"/>
+<label x="58.42" y="20.32" size="1.778" layer="95"/>
 </segment>
 </net>
@@
 </segment>
 <segment>
-<pinref part="JP3" gate="G$1" pin="1"/>
-<wire x1="73.66" y1="22.86" x2="66.04" y2="22.86" width="0.1524" layer="91"/>
-<label x="60.96" y="22.86" size="1.778" layer="95"/>
-</segment>
-<segment>
 <pinref part="IC1" gate="G$1" pin="OUT"/>
 <pinref part="SUPPLY6" gate="G$1" pin="VCC"/>
@@
 <label x="40.64" y="30.48" size="1.778" layer="95"/>
 </segment>
-</net>
+<segment>
+<pinref part="X2" gate="-2" pin="KL"/>
+<wire x1="66.04" y1="25.4" x2="58.42" y2="25.4" width="0.1524" layer="91"/>
+<label x="58.42" y="25.4" size="1.778" layer="95"/>
+</segment>
+</net>
